File: pcbs/transimpedance_amp/transimpedance_amp.kicad_pcb (KiCad board)
At the start: 2 copper layers, 80 x 50 mm, 48 parts, among them P1 CONN_01X05, P2 CONN_01X05, P3 CONN_01X05, P4 CONN_01X05, P5 CONN_01X05, P6 CONN_01X05, P7 CONN_01X05, P8 CONN_01X05, U1 AD8616

Commit message: Created gerber files.
Parts:
- added REF**: SolderWirePad_single_1mmDrill, Vias:Stitchging-Via-0.6, F.Cu at (174.1, 107.2)
- added REF**: SolderWirePad_single_1mmDrill, Vias:Stitchging-Via-0.6, F.Cu at (146.7, 97.0)
- added REF**: SolderWirePad_single_1mmDrill, Vias:Stitchging-Via-0.6, F.Cu at (166.6, 97.9)
- added REF**: SolderWirePad_single_1mmDrill, Vias:Stitchging-Via-0.6, F.Cu at (174.0, 84.8)
- added REF**: SolderWirePad_single_1mmDrill, Vias:Stitchging-Via-0.6, F.Cu at (130.0, 96.8)
- added REF**: SolderWirePad_single_1mmDrill, Vias:Stitchging-Via-0.6, F.Cu at (155.7, 84.8)
- added REF**: SolderWirePad_single_1mmDrill, Vias:Stitchging-Via-0.6, F.Cu at (173.2, 114.4)
- added REF**: SolderWirePad_single_1mmDrill, Vias:Stitchging-Via-0.6, F.Cu at (175.6, 116.8)
- added REF**: SolderWirePad_single_1mmDrill, Vias:Stitchging-Via-0.6, F.Cu at (165.9, 120.0)
- added REF**: SolderWirePad_single_1mmDrill, Vias:Stitchging-Via-0.6, F.Cu at (146.8, 109.9)
- added REF**: SolderWirePad_single_1mmDrill, Vias:Stitchging-Via-0.6, F.Cu at (139.3, 118.0)
- added REF**: SolderWirePad_single_1mmDrill, Vias:Stitchging-Via-0.6, F.Cu at (124.0, 124.3)
- added REF**: SolderWirePad_single_1mmDrill, Vias:Stitchging-Via-0.6, F.Cu at (118.9, 90.2)
- added REF**: SolderWirePad_single_1mmDrill, Vias:Stitchging-Via-0.6, F.Cu at (123.7, 108.7)
- REF** (x9): footprint Wire_Pads:SolderWirePad_single_1mmDrill -> Vias:Stitchging-Via-0.6
- moved REF** 2.30 mm to (148.8, 100.6)
- renumbered TP2 to 5V, TP3 to GND
Other:
- board text added: "BPW34FA"
- board text added: "Output of the BPW34 is on this side (TP4)."
- board text added: "highest current"
