File: pcbs/transimpedance_amp/transimpedance_amp.sch (KiCad schematic (older format))
At the start: 35 parts, among them P1 CONN_01X05, P2 CONN_01X05, P3 CONN_01X05, P4 CONN_01X05, P5 CONN_01X05, P6 CONN_01X05, P7 CONN_01X05, P8 CONN_01X05, U1 AD8616

Commit message: Orders for etching added.
Changed lines of the file:
@@
 	1400 4400 1400 4600
 Wire Wire Line
-	1400 4600 1550 4600
-Wire Wire Line
-	1550 4600 1700 4600
+	1400 4600 1700 4600
 Wire Wire Line
 	1700 4600 1700 4400
@@
 	1700 3900 1700 4100
 Wire Wire Line
-	1400 3900 1550 3900
-Wire Wire Line
-	1550 3900 1700 3900
+	1400 3900 1700 3900
 Wire Wire Line
 	1400 3900 1400 4100
 Wire Wire Line
-	1950 4600 2100 4600
-Wire Wire Line
-	2100 4600 2250 4600
+	1950 4600 2250 4600
 Wire Wire Line
 	2250 4600 2250 4400
@@
 	2250 3900 2250 4100
 Wire Wire Line
-	1950 3900 2100 3900
-Wire Wire Line
-	2100 3900 2250 3900
+	1950 3900 2250 3900
 Wire Wire Line
 	2500 4400 2500 4600
 Wire Wire Line
-	2500 4600 2650 4600
-Wire Wire Line
-	2650 4600 2800 4600
+	2500 4600 2800 4600
 Wire Wire Line
 	2800 4600 2800 4400
@@
 	2800 3900 2800 4100
 Wire Wire Line
-	2500 3900 2650 3900
-Wire Wire Line
-	2650 3900 2800 3900
+	2500 3900 2800 3900
 Wire Wire Line
 	2500 3900 2500 4100
@@
 	3050 4400 3050 4600
 Wire Wire Line
-	3050 4600 3200 4600
-Wire Wire Line
-	3200 4600 3350 4600
+	3050 4600 3350 4600
 Wire Wire Line
 	3350 4600 3350 4400
@@
 	3350 3900 3350 4100
 Wire Wire Line
-	3050 3900 3200 3900
-Wire Wire Line
-	3200 3900 3350 3900
+	3050 3900 3350 3900
 Wire Wire Line
 	3050 3900 3050 4100
@@
 	3550 4400 3550 4600
 Wire Wire Line
-	3550 4600 3700 4600
-Wire Wire Line
-	3700 4600 3850 4600
+	3550 4600 3850 4600
 Wire Wire Line
 	3850 4600 3850 4400
@@
 	3850 3900 3850 4100
 Wire Wire Line
-	3550 3900 3700 3900
-Wire Wire Line
-	3700 3900 3850 3900
+	3550 3900 3850 3900
 Wire Wire Line
 	3550 3900 3550 4100
 Wire Wire Line
-	2650 2850 2650 3200
-Wire Wire Line
-	2650 3200 2650 3900
+	2650 2850 2650 3900
 Connection ~ 2650 3900
 Wire Wire Line
 	2100 3900 2100 3800
 Wire Wire Line
-	2100 3800 2550 3800
-Wire Wire Line
-	2550 3800 2550 3100
-Wire Wire Line
-	2550 3100 2550 2850
+	2550 3800 2100 3800
+Wire Wire Line
+	2550 2850 2550 3800
 Connection ~ 2100 3900
 Wire Wire Line
-	2450 2850 2450 3000
-Wire Wire Line
-	2450 3000 2450 3700
+	2450 2850 2450 3700
 Wire Wire Line
 	2450 3700 1550 3700
 Wire Wire Line
-	2750 2850 2750 3300
-Wire Wire Line
-	2750 3300 2750 3800
-Wire Wire Line
-	2850 2850 2850 3400
-Wire Wire Line
-	2850 3400 2850 3700
+	2750 2850 2750 3800
+Wire Wire Line
+	2850 2850 2850 3700
 Wire Wire Line
 	5050 4350 4950 4350
@@
 	4950 4350 4950 5200
 Wire Wire Line
-	4050 4150 4400 4150
-Wire Wire Line
-	4400 4150 5050 4150
+	4050 4150 5050 4150
 Wire Wire Line
 	4400 5200 4400 4700
 Wire Wire Line
-	4400 3000 4400 3100
-Wire Wire Line
-	4400 3100 4400 3200
-Wire Wire Line
-	4400 3200 4400 3300
-Wire Wire Line
-	4400 3300 4400 3400
+	4400 3000 4400 3400
 Connection ~ 4400 3100
 Connection ~ 4400 3200
@@
 	3700 3700 3700 3900
 Wire Wire Line
-	2450 2150 2550 2150
-Wire Wire Line
-	2550 2150 2650 2150
-Wire Wire Line
-	2650 2150 2750 2150
-Wire Wire Line
-	2750 2150 2850 2150
-Wire Wire Line
-	2850 2150 4900 2150
+	2450 2150 4900 2150
 Wire Wire Line
 	4900 2150 4900 3950
@@
 	10250 4600 10250 4400
 Wire Wire Line
-	9950 4600 10100 4600
-Wire Wire Line
-	10100 4600 10250 4600
+	9950 4600 10250 4600
 Wire Wire Line
 	9950 4600 9950 4400
@@
 	9950 3900 9950 4100
 Wire Wire Line
-	9950 3900 10100 3900
-Wire Wire Line
-	10100 3900 10250 3900
+	9950 3900 10250 3900
 Wire Wire Line
 	10250 3900 10250 4100
 Wire Wire Line
-	9400 4600 9550 4600
-Wire Wire Line
-	9550 4600 9700 4600
+	9400 4600 9700 4600
 Wire Wire Line
 	9400 4600 9400 4400
@@
 	9400 3900 9400 4100
 Wire Wire Line
-	9400 3900 9550 3900
-Wire Wire Line
-	9550 3900 9700 3900
+	9400 3900 9700 3900
 Wire Wire Line
 	9150 4600 9150 4400
 Wire Wire Line
-	8850 4600 9000 4600
-Wire Wire Line
-	9000 4600 9150 4600
+	8850 4600 9150 4600
 Wire Wire Line
 	8850 4600 8850 4400
@@
 	8850 3900 8850 4100
 Wire Wire Line
-	8850 3900 9000 3900
-Wire Wire Line
-	9000 3900 9150 3900
+	8850 3900 9150 3900
 Wire Wire Line
 	9150 3900 9150 4100
@@
 	8600 4600 8600 4400
 Wire Wire Line
-	8300 4600 8450 4600
-Wire Wire Line
-	8450 4600 8600 4600
+	8300 4600 8600 4600
 Wire Wire Line
 	8300 4600 8300 4400
@@
 	8300 3900 8300 4100
 Wire Wire Line
-	8300 3900 8450 3900
-Wire Wire Line
-	8450 3900 8600 3900
+	8300 3900 8600 3900
 Wire Wire Line
 	8600 3900 8600 4100
@@
 	8100 4600 8100 4400
 Wire Wire Line
-	7800 4600 7950 4600
-Wire Wire Line
-	7950 4600 8100 4600
+	7800 4600 8100 4600
 Wire Wire Line
 	7800 4600 7800 4400
@@
 	7800 3900 7800 4100
 Wire Wire Line
-	7800 3900 7950 3900
-Wire Wire Line
-	7950 3900 8100 3900
+	7800 3900 8100 3900
 Wire Wire Line
 	8100 3900 8100 4100
 Wire Wire Line
-	9000 2850 9000 3200
-Wire Wire Line
-	9000 3200 9000 3900
+	9000 2850 9000 3900
 Connection ~ 9000 3900
 Wire Wire Line
 	9550 3900 9550 3800
 Wire Wire Line
-	9550 3800 9100 3800
-Wire Wire Line
-	9100 3800 9100 3100
-Wire Wire Line
-	9100 3100 9100 2850
+	9100 3800 9550 3800
+Wire Wire Line
+	9100 2850 9100 3800
 Connection ~ 9550 3900
 Wire Wire Line
-	9200 2850 9200 3000
-Wire Wire Line
-	9200 3000 9200 3700
+	9200 2850 9200 3700
 Wire Wire Line
 	9200 3700 10100 3700
 Wire Wire Line
-	8900 2850 8900 3300
-Wire Wire Line
-	8900 3300 8900 3800
-Wire Wire Line
-	8800 2850 8800 3400
-Wire Wire Line
-	8800 3400 8800 3700
-Wire Wire Line
-	6600 4150 7250 4150
-Wire Wire Line
-	7250 4150 7600 4150
+	8900 2850 8900 3800
+Wire Wire Line
+	8800 2850 8800 3700
+Wire Wire Line
+	6600 4150 7600 4150
 Wire Wire Line
 	7250 5200 7250 4700
 Wire Wire Line
-	7250 3000 7250 3100
-Wire Wire Line
-	7250 3100 7250 3200
-Wire Wire Line
-	7250 3200 7250 3300
-Wire Wire Line
-	7250 3300 7250 3400
+	7250 3000 7250 3400
 Connection ~ 7250 3100
 Connection ~ 7250 3200
@@
 	7950 3700 7950 3900
 Wire Wire Line
-	6750 2150 8800 2150
-Wire Wire Line
-	8800 2150 8900 2150
-Wire Wire Line
-	8900 2150 9000 2150
-Wire Wire Line
-	9000 2150 9100 2150
-Wire Wire Line
-	9100 2150 9200 2150
+	6750 2150 9200 2150
 Wire Wire Line
 	6750 2150 6750 3950
@@
 	6050 2450 6050 2600
 Wire Wire Line
-	1550 5200 2100 5200
-Wire Wire Line
-	2100 5200 2650 5200
-Wire Wire Line
-	2650 5200 3200 5200
-Wire Wire Line
-	3200 5200 3700 5200
-Wire Wire Line
-	3700 5200 4050 5200
+	1550 5200 4050 5200
 Wire Wire Line
 	4050 5200 4050 4150
 Connection ~ 4400 4150
 Wire Wire Line
-	7600 5200 7950 5200
-Wire Wire Line
-	7950 5200 8450 5200
-Wire Wire Line
-	8450 5200 9000 5200
-Wire Wire Line
-	9000 5200 9550 5200
-Wire Wire Line
-	9550 5200 10100 5200
+	7600 5200 10100 5200
 Wire Wire Line
 	7600 4150 7600 5200
