File: pcbs/analog_board_v0.2/_autosave-analog_board_v0.2.kicad_pcb (KiCad board)
At the start: 2 copper layers, 80 x 50 mm, 95 parts, among them J1 CONN_02X03, J2 CONN_02X07, J3 CONN_01X04, P1 CONN_01X03, P2 CONN_01X03, P3 CONN_01X03, Q1 DMP2035U, Q2 TSM2314, Q3 DMP2035U, Q4 TSM2314, Q5 DMP2035U, Q6 TSM2314, Q7 DMP2035U, Q8 TSM2314, Q9 MMBT3904, U1 ADA4530-1, U2 ADA4522-2, U3 ICL7660S, U4 AD8616

Commit message: Added some iportant backplane spec.
Connections:
- J1 pad 1: +5V -> GND
- J1 pad 2: GND -> +5V
- J1 pad 3: /interface/ADC1 -> /interface/ADC3
- J1 pad 4: /interface/ADC3 -> /interface/ADC1
- J1 pad 5: /interface/ADC2 -> /interface/ADC4
- J1 pad 6: /interface/ADC4 -> /interface/ADC2
Changed lines of the file:
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@@
     (fp_line (start 12.7 -1.6) (end -1.6 -1.6) (layer F.CrtYd) (width 0.05))
     (pad 1 thru_hole rect (at 0 0 90) (size 1.7 1.7) (drill 1) (layers *.Cu *.Mask)
+      (net 2 GND))
+    (pad 2 thru_hole oval (at 2.54 0 90) (size 1.7 1.7) (drill 1) (layers *.Cu *.Mask)
       (net 11 +5V))
-    (pad 2 thru_hole oval (at 2.54 0 90) (size 1.7 1.7) (drill 1) (layers *.Cu *.Mask)
-      (net 2 GND))
     (pad 3 thru_hole oval (at 0 2.54 90) (size 1.7 1.7) (drill 1) (layers *.Cu *.Mask)
+      (net 8 /interface/ADC3))
+    (pad 4 thru_hole oval (at 2.54 2.54 90) (size 1.7 1.7) (drill 1) (layers *.Cu *.Mask)
       (net 6 /interface/ADC1))
-    (pad 4 thru_hole oval (at 2.54 2.54 90) (size 1.7 1.7) (drill 1) (layers *.Cu *.Mask)
-      (net 8 /interface/ADC3))
     (pad 5 thru_hole oval (at 0 5.08 90) (size 1.7 1.7) (drill 1) (layers *.Cu *.Mask)
+      (net 13 /interface/ADC4))
+    (pad 6 thru_hole oval (at 2.54 5.08 90) (size 1.7 1.7) (drill 1) (layers *.Cu *.Mask)
       (net 7 /interface/ADC2))
-    (pad 6 thru_hole oval (at 2.54 5.08 90) (size 1.7 1.7) (drill 1) (layers *.Cu *.Mask)
-      (net 13 /interface/ADC4))
     (model Pin_Headers.3dshapes/Pin_Header_Angled_2x03_Pitch2.54mm.wrl
       (at (xyz 0.05 -0.1 0))
