File: pcbs/analog_board_v0.2/highCurrentPart.sch (KiCad schematic (older format))
At the start: 36 parts, among them J3 CONN_01X04, P1 CONN_01X03, P2 CONN_01X03, P3 CONN_01X03, Q1 DMP2035U, Q2 TSM2314, Q3 DMP2035U, Q4 TSM2314, Q5 DMP2035U, Q6 TSM2314, Q7 DMP2035U, Q8 TSM2314, Q9 MMBT3904, U3 ICL7660S, U4 AD8616

Commit message: Added BOMs and gerber files.
Parts:
- Q2, Q4, Q6, Q8: Farnell TSM2314CX -> 1864589
- Q9: Farnell 1757936RL -> 1757935
- R9: Farnell 2504961 -> 1632456
- U3: Farnell ICL7660SCBAZ -> 1561969
- U4: Farnell AD8616ARZ -> 1581952
Other:
- note added: "Investigate if AD8616 here can be replaced by the LM358 (most likely yes, footprints match)."
Changed lines of the file:
@@
 $EndDescr
 $Comp
-L GND #PWR36
+L GND #PWR018
 U 1 1 5940A4E3
 P 8150 3325
-F 0 "#PWR36" H 8150 3075 50  0001 C CNN
+F 0 "#PWR018" H 8150 3075 50  0001 C CNN
 F 1 "GND" H 8150 3175 50  0000 C CNN
 F 2 "" H 8150 3325 50  0000 C CNN
@@
 F 2 "SMD_Packages:SOIC-8-N" H 7953 2700 50  0001 C CNN
 F 3 "http://www.farnell.com/datasheets/1841629.pdf" H 7853 2800 50  0001 C CNN
-F 4 "AD8616ARZ" H 8150 2650 60  0001 C CNN "Farnell"
+F 4 "1581952" H 8150 2650 60  0001 C CNN "Farnell"
 	1    8150 2650
 	1    0    0    -1
@@
 $EndComp
 $Comp
-L GND #PWR41
+L GND #PWR019
 U 1 1 5940A554
 P 9725 3325
-F 0 "#PWR41" H 9725 3075 50  0001 C CNN
+F 0 "#PWR019" H 9725 3075 50  0001 C CNN
 F 1 "GND" H 9725 3175 50  0000 C CNN
 F 2 "" H 9725 3325 50  0000 C CNN
@@
 F 2 "Resistors_SMD:R_0805" V 6705 3075 50  0001 C CNN
 F 3 "" H 6775 3075 50  0000 C CNN
-F 4 "2504961" V 6775 3075 60  0001 C CNN "Farnell"
+F 4 "1632456" V 6775 3075 60  0001 C CNN "Farnell"
 	1    6775 3075
 	1    0    0    -1
@@
 	6775 2050 6775 2150
 $Comp
-L +5V #PWR31
+L +5V #PWR020
 U 1 1 5940A5DC
 P 6775 1675
-F 0 "#PWR31" H 6775 1525 50  0001 C CNN
+F 0 "#PWR020" H 6775 1525 50  0001 C CNN
 F 1 "+5V" H 6775 1815 50  0000 C CNN
 F 2 "" H 6775 1675 50  0000 C CNN
@@
 	6775 1675 6775 1750
 $Comp
-L GND #PWR32
+L GND #PWR021
 U 1 1 5940A5E4
 P 6775 3350
-F 0 "#PWR32" H 6775 3100 50  0001 C CNN
+F 0 "#PWR021" H 6775 3100 50  0001 C CNN
 F 1 "GND" H 6775 3200 50  0000 C CNN
 F 2 "" H 6775 3350 50  0000 C CNN
@@
 F 2 "TO_SOT_Packages_SMD:SOT-23" H 7075 2275 50  0001 L CIN
 F 3 "https://www.fairchildsemi.com/datasheets/MM/MMBT3904.pdf" H 6875 2350 50  0001 L CNN
-F 4 "1757936RL" H 6875 2350 60  0001 C CNN "Farnell"
+F 4 "1757935" H 6875 2350 60  0001 C CNN "Farnell"
 	1    6875 2350
 	-1   0    0    -1
@@
 Signal
 $Comp
-L GND #PWR34
+L GND #PWR022
 U 1 1 5940A601
 P 7675 3925
-F 0 "#PWR34" H 7675 3675 50  0001 C CNN
+F 0 "#PWR022" H 7675 3675 50  0001 C CNN
 F 1 "GND" H 7675 3775 50  0000 C CNN
 F 2 "" H 7675 3925 50  0000 C CNN
@@
 Signal
 $Comp
-L +5V #PWR38
+L +5V #PWR023
 U 1 1 5940A60A
 P 8450 3925
-F 0 "#PWR38" H 8450 3775 50  0001 C CNN
+F 0 "#PWR023" H 8450 3775 50  0001 C CNN
 F 1 "+5V" H 8450 4065 50  0000 C CNN
 F 2 "" H 8450 3925 50  0000 C CNN
@@
 Connection ~ 6775 2775
 $Comp
-L GND #PWR39
+L GND #PWR024
 U 1 1 5940EF10
 P 8900 3325
-F 0 "#PWR39" H 8900 3075 50  0001 C CNN
+F 0 "#PWR024" H 8900 3075 50  0001 C CNN
 F 1 "GND" H 8900 3175 50  0000 C CNN
 F 2 "" H 8900 3325 50  0000 C CNN
@@
 Connection ~ 7600 1600
 $Comp
-L GND #PWR33
+L GND #PWR025
 U 1 1 594122F3
 P 7350 1975
-F 0 "#PWR33" H 7350 1725 50  0001 C CNN
+F 0 "#PWR025" H 7350 1725 50  0001 C CNN
 F 1 "GND" H 7350 1825 50  0000 C CNN
 F 2 "" H 7350 1975 50  0000 C CNN
@@
 $EndComp
 $Comp
-L +5V #PWR40
+L +5V #PWR026
 U 1 1 5941842E
 P 9075 4125
-F 0 "#PWR40" H 9075 3975 50  0001 C CNN
+F 0 "#PWR026" H 9075 3975 50  0001 C CNN
 F 1 "+5V" H 9075 4265 50  0000 C CNN
 F 2 "" H 9075 4125 50  0000 C CNN
@@
 	8600 4125 8750 4125
 $Comp
-L GND #PWR37
+L GND #PWR027
 U 1 1 5941869D
 P 8225 4125
-F 0 "#PWR37" H 8225 3875 50  0001 C CNN
+F 0 "#PWR027" H 8225 3875 50  0001 C CNN
 F 1 "GND" H 8225 3975 50  0000 C CNN
 F 2 "" H 8225 4125 50  0000 C CNN
@@
 BPW34_OUT
 $Comp
-L GND #PWR26
+L GND #PWR028
 U 1 1 59553CC6
 P 3000 1800
-F 0 "#PWR26" H 3000 1550 50  0001 C CNN
+F 0 "#PWR028" H 3000 1550 50  0001 C CNN
 F 1 "GND" H 3000 1650 50  0000 C CNN
 F 2 "" H 3000 1800 50  0001 C CNN
@@
 	1    0    0    1
 $EndComp
-$Comp
-L Q_NMOS_GSD Q4
-U 1 1 59557415
-P 2275 6125
-F 0 "Q4" H 2475 6175 50  0000 L CNN
-F 1 "TSM2314" H 2475 6075 50  0000 L CNN
-F 2 "TO_SOT_Packages_SMD:SOT-23" H 2475 6225 50  0001 C CNN
-F 3 "http://www.farnell.com/datasheets/2044480.pdf" H 2275 6125 50  0001 C CNN
-F 4 "TSM2314CX" H 2275 6125 60  0001 C CNN "Farnell"
-	1    2275 6125
-	1    0    0    -1
-$EndComp
 Wire Wire Line
 	2375 5675 2375 5925
 $Comp
-L GND #PWR23
+L GND #PWR029
 U 1 1 59557860
 P 2375 6425
-F 0 "#PWR23" H 2375 6175 50  0001 C CNN
+F 0 "#PWR029" H 2375 6175 50  0001 C CNN
 F 1 "GND" H 2375 6275 50  0000 C CNN
 F 2 "" H 2375 6425 50  0000 C CNN
@@
 	2375 6325 2375 6425
 $Comp
-L +5V #PWR22
+L +5V #PWR030
 U 1 1 59557DF9
 P 2375 5200
-F 0 "#PWR22" H 2375 5050 50  0001 C CNN
+F 0 "#PWR030" H 2375 5050 50  0001 C CNN
 F 1 "+5V" H 2375 5340 50  0000 C CNN
 F 2 "" H 2375 5200 50  0000 C CNN
@@
 	4025 5675 4025 5925
 $Comp
-L GND #PWR30
+L GND #PWR031
 U 1 1 59558304
 P 4025 6425
-F 0 "#PWR30" H 4025 6175 50  0001 C CNN
+F 0 "#PWR031" H 4025 6175 50  0001 C CNN
 F 1 "GND" H 4025 6275 50  0000 C CNN
 F 2 "" H 4025 6425 50  0000 C CNN
@@
 	4025 6325 4025 6425
 $Comp
-L +5V #PWR29
+L +5V #PWR032
 U 1 1 5955830B
 P 4025 5200
-F 0 "#PWR29" H 4025 5050 50  0001 C CNN
+F 0 "#PWR032" H 4025 5050 50  0001 C CNN
 F 1 "+5V" H 4025 5340 50  0000 C CNN
 F 2 "" H 4025 5200 50  0000 C CNN
@@
 	4525 5800 4450 5800
 Connection ~ 4450 5800
-$Comp
-L Q_NMOS_GSD Q8
-U 1 1 59558B41
-P 4125 6125
-F 0 "Q8" H 4325 6175 50  0000 L CNN
-F 1 "TSM2314" H 4325 6075 50  0000 L CNN
-F 2 "TO_SOT_Packages_SMD:SOT-23" H 4325 6225 50  0001 C CNN
-F 3 "http://www.farnell.com/datasheets/2044480.pdf" H 4125 6125 50  0001 C CNN
-F 4 "TSM2314CX" H 4125 6125 60  0001 C CNN "Farnell"
-	1    4125 6125
-	-1   0    0    -1
-$EndComp
 $Comp
 L Q_PMOS_GSD Q7
@@
 F 2 "TO_SOT_Packages_SMD:SOT-23" H 2475 4525 50  0001 C CNN
 F 3 "http://www.farnell.com/datasheets/2044480.pdf" H 2275 4425 50  0001 C CNN
-F 4 "TSM2314CX" H 2275 4425 60  0001 C CNN "Farnell"
+F 4 "1864589" H 2275 4425 60  0001 C CNN "Farnell"
 	1    2275 4425
 	1    0    0    -1
@@
 	2375 3975 2375 4225
 $Comp
-L GND #PWR21
+L GND #PWR033
 U 1 1 5956291A
 P 2375 4725
-F 0 "#PWR21" H 2375 4475 50  0001 C CNN
+F 0 "#PWR033" H 2375 4475 50  0001 C CNN
 F 1 "GND" H 2375 4575 50  0000 C CNN
 F 2 "" H 2375 4725 50  0000 C CNN
@@
 	2375 4625 2375 4725
 $Comp
-L +5V #PWR20
+L +5V #PWR034
 U 1 1 59562921
 P 2375 3500
-F 0 "#PWR20" H 2375 3350 50  0001 C CNN
+F 0 "#PWR034" H 2375 3350 50  0001 C CNN
 F 1 "+5V" H 2375 3640 50  0000 C CNN
 F 2 "" H 2375 3500 50  0000 C CNN
@@
 	4025 3975 4025 4225
 $Comp
-L GND #PWR28
+L GND #PWR035
 U 1 1 59562931
 P 4025 4725
-F 0 "#PWR28" H 4025 4475 50  0001 C CNN
+F 0 "#PWR035" H 4025 4475 50  0001 C CNN
 F 1 "GND" H 4025 4575 50  0000 C CNN
 F 2 "" H 4025 4725 50  0000 C CNN
@@
 	4025 4625 4025 4725
 $Comp
-L +5V #PWR27
+L +5V #PWR036
 U 1 1 59562938
 P 4025 3500
-F 0 "#PWR27" H 4025 3350 50  0001 C CNN
+F 0 "#PWR036" H 4025 3350 50  0001 C CNN
 F 1 "+5V" H 4025 3640 50  0000 C CNN
 F 2 "" H 4025 3500 50  0000 C CNN
@@
 	4525 4100 4450 4100
 Connection ~ 4450 4100
-$Comp
-L Q_NMOS_GSD Q6
-U 1 1 5956294D
-P 4125 4425
-F 0 "Q6" H 4325 4475 50  0000 L CNN
-F 1 "TSM2314" H 4325 4375 50  0000 L CNN
-F 2 "TO_SOT_Packages_SMD:SOT-23" H 4325 4525 50  0001 C CNN
-F 3 "http://www.farnell.com/datasheets/2044480.pdf" H 4125 4425 50  0001 C CNN
-F 4 "TSM2314CX" H 4125 4425 60  0001 C CNN "Farnell"
-	1    4125 4425
-	-1   0    0    -1
-$EndComp
 $Comp
 L Q_PMOS_GSD Q5
@@
 LED_CONTROLL
 $Comp
-L GND #PWR19
+L GND #PWR037
 U 1 1 59563916
 P 1850 1800
-F 0 "#PWR19" H 1850 1550 50  0001 C CNN
+F 0 "#PWR037" H 1850 1550 50  0001 C CNN
 F 1 "GND" H 1850 1650 50  0000 C CNN
 F 2 "" H 1850 1800 50  0001 C CNN
@@
 	2000 2025 2000 1950
 $Comp
-L +3.3V #PWR25
+L +3.3V #PWR038
 U 1 1 59563EC0
 P 3000 1425
-F 0 "#PWR25" H 3000 1275 50  0001 C CNN
+F 0 "#PWR038" H 3000 1275 50  0001 C CNN
 F 1 "+3.3V" H 3000 1565 50  0000 C CNN
 F 2 "" H 3000 1425 50  0001 C CNN
@@
 	2900 1950 2900 2100
 $Comp
-L GND #PWR24
+L GND #PWR039
 U 1 1 5956469D
 P 2900 2425
-F 0 "#PWR24" H 2900 2175 50  0001 C CNN
+F 0 "#PWR039" H 2900 2175 50  0001 C CNN
 F 1 "GND" H 2900 2275 50  0000 C CNN
 F 2 "" H 2900 2425 50  0001 C CNN
@@
 $EndComp
 $Comp
-L +3.3V #PWR18
+L +3.3V #PWR040
 U 1 1 595680C2
 P 1825 1125
-F 0 "#PWR18" H 1825 975 50  0001 C CNN
+F 0 "#PWR040" H 1825 975 50  0001 C CNN
 F 1 "+3.3V" H 1825 1265 50  0000 C CNN
 F 2 "" H 1825 1125 50  0001 C CNN
@@
 F 2 "SMD_Packages:SOIC-8-N" H 2400 1500 60  0001 C CNN
 F 3 "http://www.farnell.com/datasheets/2059962.pdf" H 2400 1500 60  0001 C CNN
-F 4 "ICL7660SCBAZ" H 2400 1500 60  0001 C CNN "Farnell"
+F 4 "1561969" H 2400 1500 60  0001 C CNN "Farnell"
 	1    2400 1500
 	1    0    0    -1
@@
 Low-pass has a cut-off freq. of approx. 1.6 Hz, ergo DC.
 $Comp
-L +3.3V #PWR35
+L +3.3V #PWR041
 U 1 1 595BE0DA
 P 8150 1525
-F 0 "#PWR35" H 8150 1375 50  0001 C CNN
+F 0 "#PWR041" H 8150 1375 50  0001 C CNN
 F 1 "+3.3V" H 8150 1665 50  0000 C CNN
 F 2 "" H 8150 1525 50  0001 C CNN
@@
 	-1   0    0    -1
 $EndComp
+$Comp
+L Q_NMOS_GSD Q4
+U 1 1 59557415
+P 2275 6125
+F 0 "Q4" H 2475 6175 50  0000 L CNN
+F 1 "TSM2314" H 2475 6075 50  0000 L CNN
+F 2 "TO_SOT_Packages_SMD:SOT-23" H 2475 6225 50  0001 C CNN
+F 3 "http://www.farnell.com/datasheets/2044480.pdf" H 2275 6125 50  0001 C CNN
+F 4 "1864589" H 2275 6125 60  0001 C CNN "Farnell"
+	1    2275 6125
+	1    0    0    -1
+$EndComp
+$Comp
+L Q_NMOS_GSD Q8
+U 1 1 59558B41
+P 4125 6125
+F 0 "Q8" H 4325 6175 50  0000 L CNN
+F 1 "TSM2314" H 4325 6075 50  0000 L CNN
+F 2 "TO_SOT_Packages_SMD:SOT-23" H 4325 6225 50  0001 C CNN
+F 3 "http://www.farnell.com/datasheets/2044480.pdf" H 4125 6125 50  0001 C CNN
+F 4 "1864589" H 4125 6125 60  0001 C CNN "Farnell"
+	1    4125 6125
+	-1   0    0    -1
+$EndComp
+$Comp
+L Q_NMOS_GSD Q6
+U 1 1 5956294D
+P 4125 4425
+F 0 "Q6" H 4325 4475 50  0000 L CNN
+F 1 "TSM2314" H 4325 4375 50  0000 L CNN
+F 2 "TO_SOT_Packages_SMD:SOT-23" H 4325 4525 50  0001 C CNN
+F 3 "http://www.farnell.com/datasheets/2044480.pdf" H 4125 4425 50  0001 C CNN
+F 4 "1864589" H 4125 4425 60  0001 C CNN "Farnell"
+	1    4125 4425
+	-1   0    0    -1
+$EndComp
+Text Notes 5550 3700 0    60   ~ 0
+Investigate if AD8616 here can be replaced by the LM358 (most likely yes, footprints match).
 $EndSCHEMATC

Commit message: Mechanics developed further.
Other:
- note added: "Constant current source with 100R sensing resistor. Monitoring diode included\nwith 1mA being translated into 1V.\n"
- note removed: "Constant current source with 100R sensing resistor. Monitoring diode included\nwith 1uA being translated into 1V.\n"
Changed lines of the file:
@@
 	7900 4450 9000 4450
 Text Notes 6425 5175 0    60   ~ 0
-Constant current source with 100R sensing resistor. Monitoring diode included\nwith 1uA being translated into 1V.\n
+Constant current source with 100R sensing resistor. Monitoring diode included\nwith 1mA being translated into 1V.\n
 Text Notes 8650 3800 0    60   ~ 0
 Constant current with ca. 4.55 mA.
