File: pcbs/analog_board_v0.22/analog_board_v0.22.sch (KiCad schematic (older format))
At the start: 3 parts

Commit message: Mechanics developed further.
Changed lines of the file:
@@
 $EndSheet
 $Comp
-L +3.3V #PWR01
-U 1 1 59551FE0
-P 4475 3125
-F 0 "#PWR01" H 4475 2975 50  0001 C CNN
-F 1 "+3.3V" H 4475 3265 50  0000 C CNN
-F 2 "" H 4475 3125 50  0001 C CNN
-F 3 "" H 4475 3125 50  0001 C CNN
-	1    4475 3125
-	1    0    0    -1
-$EndComp
-Wire Wire Line
-	4825 3125 4475 3125
-$Comp
-L GND #PWR02
+L GND #PWR01
 U 1 1 595520F8
 P 4475 3225
-F 0 "#PWR02" H 4475 2975 50  0001 C CNN
+F 0 "#PWR01" H 4475 2975 50  0001 C CNN
 F 1 "GND" H 4475 3075 50  0000 C CNN
 F 2 "" H 4475 3225 50  0001 C CNN
@@
 $EndComp
 Wire Wire Line
-	4475 3225 4825 3225
+	4125 3225 4825 3225
 $Comp
-L +5V #PWR03
+L +5V #PWR02
 U 1 1 59552732
-P 4475 2875
-F 0 "#PWR03" H 4475 2725 50  0001 C CNN
-F 1 "+5V" H 4475 3015 50  0000 C CNN
-F 2 "" H 4475 2875 50  0001 C CNN
-F 3 "" H 4475 2875 50  0001 C CNN
-	1    4475 2875
+P 4475 2850
+F 0 "#PWR02" H 4475 2700 50  0001 C CNN
+F 1 "+5V" H 4475 2990 50  0000 C CNN
+F 2 "" H 4475 2850 50  0001 C CNN
+F 3 "" H 4475 2850 50  0001 C CNN
+	1    4475 2850
 	1    0    0    -1
 $EndComp
@@
 	4825 3025 4625 3025
 Wire Wire Line
-	4625 3025 4625 2875
+	4625 2875 4625 3025
 Wire Wire Line
-	4625 2875 4475 2875
+	4125 2875 4625 2875
 Wire Wire Line
 	7675 3025 6525 3025
@@
 	1375 3175 1850 3175
 $Comp
-L +3.3V #PWR04
+L +3.3V #PWR03
 U 1 1 59593859
 P 1500 3025
-F 0 "#PWR04" H 1500 2875 50  0001 C CNN
+F 0 "#PWR03" H 1500 2875 50  0001 C CNN
 F 1 "+3.3V" H 1500 3165 50  0000 C CNN
 F 2 "" H 1500 3025 50  0001 C CNN
@@
 Wire Wire Line
 	4525 3825 4825 3825
+$Comp
+L PWR_FLAG #FLG04
+U 1 1 5960DA74
+P 4125 2875
+F 0 "#FLG04" H 4125 2950 50  0001 C CNN
+F 1 "PWR_FLAG" H 4125 3025 50  0000 C CNN
+F 2 "" H 4125 2875 50  0001 C CNN
+F 3 "" H 4125 2875 50  0001 C CNN
+	1    4125 2875
+	1    0    0    -1
+$EndComp
+Connection ~ 4475 2875
+Wire Wire Line
+	4475 2850 4475 2875
+Wire Wire Line
+	4475 3100 4475 3125
+$Comp
+L +3.3V #PWR05
+U 1 1 59551FE0
+P 4475 3100
+F 0 "#PWR05" H 4475 2950 50  0001 C CNN
+F 1 "+3.3V" H 4475 3240 50  0000 C CNN
+F 2 "" H 4475 3100 50  0001 C CNN
+F 3 "" H 4475 3100 50  0001 C CNN
+	1    4475 3100
+	1    0    0    -1
+$EndComp
+Wire Wire Line
+	4475 3125 4825 3125
+$Comp
+L PWR_FLAG #FLG06
+U 1 1 5960F53C
+P 4125 3225
+F 0 "#FLG06" H 4125 3300 50  0001 C CNN
+F 1 "PWR_FLAG" H 4125 3375 50  0000 C CNN
+F 2 "" H 4125 3225 50  0001 C CNN
+F 3 "" H 4125 3225 50  0001 C CNN
+	1    4125 3225
+	1    0    0    -1
+$EndComp
+Connection ~ 4475 3225
 $EndSCHEMATC
