File: pcbs/analog_board_v0.22/analog_board_v0.22.sch (KiCad schematic (older format))
At the start: 4 parts

Commit message: Ananlog v0.33 is ready.
Parts:
- removed TP2: DAC1, Tespoints:TP_SMD_quadr_1mm, symbol TEST
Other:
- note removed: "Battery monitoring."
Changed lines of the file:
@@
 LIBS:ada4522-2
 LIBS:ltc6268
-LIBS:analog_board_v0.33-cache
+LIBS:analog_board_v0.22-cache
 EELAYER 25 0
 EELAYER END
@@
 Sheet 1 4
 Title "SensUs Sensor Board"
-Date "2017-08-20"
-Rev "v.0.3"
+Date "2017-07-05"
+Rev "v.0.2"
 Comp "UppSense Heart Failure Diagnostics"
 Comment1 ""
@@
 F0 "sensitiveReadout" 60
 F1 "sensitiveReadout.sch" 60
-F2 "V_SENS_NEG" I L 1850 3275 60
-F3 "V_SENS_POS" I L 1850 3150 60
-F4 "BPWFA_OUT" O R 3550 3525 60
-F5 "BPWFA_OUT_AMP" O R 3550 3625 60
+F2 "-3.3V" I L 1850 3175 60
+F3 "3.3V" I L 1850 3025 60
+F4 "BPWFA_OUT_X1" O R 3550 3525 60
+F5 "BPWFA_OUT_X100" O R 3550 3625 60
+F6 "BPWFA_OUT_X1000" O R 3550 3725 60
 $EndSheet
 $Sheet
@@
 F10 "DAC1" O R 6525 3025 60
 F11 "DAC2" O R 6525 3125 60
-F12 "I2C_SDA" B R 6525 3825 60
+F12 "GPIO4" B R 6525 3575 60
+F13 "GPIO3" B R 6525 3475 60
+F14 "GPIO2" B R 6525 3375 60
+F15 "GPIO1" B R 6525 3275 60
+F16 "I2C_SDA" B R 6525 3825 60
 $EndSheet
 $Sheet
@@
 F1 "highCurrentPart.sch" 60
 F2 "BPW34_OUT" O R 9375 3950 60
-F3 "LED_CONTROLL" I L 7675 3025 60
-F4 "V_SENS_POS" O R 9375 3575 60
-F5 "V_SENS_NEG" O R 9375 3700 60
+F3 "GPIO_COIL_3" I L 7675 3475 60
+F4 "GPIO_COIL_4" I L 7675 3575 60
+F5 "GPIO_COIL_1" I L 7675 3275 60
+F6 "GPIO_COIL_2" I L 7675 3375 60
+F7 "LED_CONTROLL" I L 7675 3025 60
+F8 "-3.3V" O R 9375 3825 60
 $EndSheet
 $Comp
-L +5V #PWR01
+L GND #PWR01
+U 1 1 595520F8
+P 4475 3225
+F 0 "#PWR01" H 4475 2975 50  0001 C CNN
+F 1 "GND" H 4475 3075 50  0000 C CNN
+F 2 "" H 4475 3225 50  0001 C CNN
+F 3 "" H 4475 3225 50  0001 C CNN
+	1    4475 3225
+	1    0    0    -1
+$EndComp
+Wire Wire Line
+	4125 3225 4825 3225
+$Comp
+L +5V #PWR02
 U 1 1 59552732
 P 4475 2850
-F 0 "#PWR01" H 4475 2700 50  0001 C CNN
+F 0 "#PWR02" H 4475 2700 50  0001 C CNN
 F 1 "+5V" H 4475 2990 50  0000 C CNN
 F 2 "" H 4475 2850 50  0001 C CNN
@@
 Wire Wire Line
 	7675 3025 6525 3025
+Wire Wire Line
+	6525 3275 7675 3275
+Wire Wire Line
+	6525 3375 7675 3375
+Wire Wire Line
+	6525 3475 7675 3475
+Wire Wire Line
+	6525 3575 7675 3575
 $Comp
 L TEST I2C1
@@
 	3550 3525 4825 3525
 Wire Wire Line
+	3550 3625 4825 3625
+Wire Wire Line
+	3550 3725 4825 3725
+Wire Wire Line
+	9375 3825 9725 3825
+Wire Wire Line
+	9725 3825 9725 2375
+Wire Wire Line
+	9725 2375 1375 2375
+Wire Wire Line
+	1375 2375 1375 3175
+Wire Wire Line
+	1375 3175 1850 3175
+$Comp
+L +3.3V #PWR03
+U 1 1 59593859
+P 1500 3025
+F 0 "#PWR03" H 1500 2875 50  0001 C CNN
+F 1 "+3.3V" H 1500 3165 50  0000 C CNN
+F 2 "" H 1500 3025 50  0001 C CNN
+F 3 "" H 1500 3025 50  0001 C CNN
+	1    1500 3025
+	1    0    0    -1
+$EndComp
+Wire Wire Line
+	1850 3025 1500 3025
+Wire Wire Line
 	9375 3950 9725 3950
 Wire Wire Line
@@
 	4525 3825 4825 3825
 $Comp
-L PWR_FLAG #FLG02
+L PWR_FLAG #FLG04
 U 1 1 5960DA74
 P 4125 2875
-F 0 "#FLG02" H 4125 2950 50  0001 C CNN
+F 0 "#FLG04" H 4125 2950 50  0001 C CNN
 F 1 "PWR_FLAG" H 4125 3025 50  0000 C CNN
 F 2 "" H 4125 2875 50  0001 C CNN
@@
 	4475 3100 4475 3125
 $Comp
-L +3.3V #PWR03
+L +3.3V #PWR05
 U 1 1 59551FE0
 P 4475 3100
-F 0 "#PWR03" H 4475 2950 50  0001 C CNN
+F 0 "#PWR05" H 4475 2950 50  0001 C CNN
 F 1 "+3.3V" H 4475 3240 50  0000 C CNN
 F 2 "" H 4475 3100 50  0001 C CNN
@@
 $EndComp
 Wire Wire Line
-	4125 3125 4825 3125
-Wire Wire Line
-	9375 3575 9750 3575
-Wire Wire Line
-	9750 3575 9750 2175
-Wire Wire Line
-	9750 2175 1625 2175
-Wire Wire Line
-	1625 2175 1625 3150
-Wire Wire Line
-	1625 3150 1850 3150
-Wire Wire Line
-	9375 3700 10000 3700
-Wire Wire Line
-	10000 3700 10000 4525
-Wire Wire Line
-	10000 4525 1625 4525
-Wire Wire Line
-	1625 4525 1625 3275
-Wire Wire Line
-	1625 3275 1850 3275
-Wire Wire Line
-	3550 3625 4825 3625
-$Comp
-L +5V #PWR04
-U 1 1 5999F74B
-P 4475 3700
-F 0 "#PWR04" H 4475 3550 50  0001 C CNN
-F 1 "+5V" H 4475 3840 50  0000 C CNN
-F 2 "" H 4475 3700 50  0001 C CNN
-F 3 "" H 4475 3700 50  0001 C CNN
-	1    4475 3700
-	1    0    0    -1
-$EndComp
-Wire Wire Line
-	4475 3700 4475 3725
-Wire Wire Line
-	4475 3725 4825 3725
-Text Notes 3625 3800 0    60   ~ 0
-Battery monitoring.
-$Comp
-L GND #PWR05
-U 1 1 599AE9BA
-P 4475 3225
-F 0 "#PWR05" H 4475 2975 50  0001 C CNN
-F 1 "GND" H 4475 3075 50  0000 C CNN
-F 2 "" H 4475 3225 50  0001 C CNN
-F 3 "" H 4475 3225 50  0001 C CNN
-	1    4475 3225
-	1    0    0    -1
-$EndComp
-Wire Wire Line
-	4475 3225 4825 3225
+	4475 3125 4825 3125
 $Comp
 L PWR_FLAG #FLG06
-U 1 1 599B0029
-P 4125 3125
-F 0 "#FLG06" H 4125 3200 50  0001 C CNN
-F 1 "PWR_FLAG" H 4125 3275 50  0000 C CNN
-F 2 "" H 4125 3125 50  0001 C CNN
-F 3 "" H 4125 3125 50  0001 C CNN
-	1    4125 3125
-	1    0    0    -1
-$EndComp
-Connection ~ 4475 3125
-$Comp
-L TEST TP2
-U 1 1 599B1306
-P 6800 2825
-F 0 "TP2" H 6800 3125 50  0000 C BNN
-F 1 "DAC1" H 6800 3075 50  0000 C CNN
-F 2 "Tespoints:TP_SMD_quadr_1mm" H 6800 2825 50  0001 C CNN
-F 3 "" H 6800 2825 50  0001 C CNN
-	1    6800 2825
-	0    1    1    0
-$EndComp
-Wire Wire Line
-	6800 2825 6675 2825
-Wire Wire Line
-	6675 2825 6675 3025
-Connection ~ 6675 3025
+U 1 1 5960F53C
+P 4125 3225
+F 0 "#FLG06" H 4125 3300 50  0001 C CNN
+F 1 "PWR_FLAG" H 4125 3375 50  0000 C CNN
+F 2 "" H 4125 3225 50  0001 C CNN
+F 3 "" H 4125 3225 50  0001 C CNN
+	1    4125 3225
+	1    0    0    -1
+$EndComp
+Connection ~ 4475 3225
 $EndSCHEMATC

Commit message: Worked on the analog PCB v0.33.
Changed lines of the file:
@@
 F6 "GPIO_COIL_2" I L 7675 3375 60
 F7 "LED_CONTROLL" I L 7675 3025 60
-F8 "-3.3V" O R 9375 3825 60
+F8 "V_SENS_POS" O R 9375 3575 60
+F9 "V_SENS_NEG" O R 9375 3700 60
 $EndSheet
 $Comp
@@
 Wire Wire Line
 	3550 3725 4825 3725
-Wire Wire Line
-	9375 3825 9725 3825
-Wire Wire Line
-	9725 3825 9725 2375
-Wire Wire Line
-	9725 2375 1375 2375
-Wire Wire Line
-	1375 2375 1375 3175
-Wire Wire Line
-	1375 3175 1850 3175
 $Comp
 L +3.3V #PWR03
