File: pcbs/analog_board_v0.22/analog_board_v0.22.kicad_pcb (KiCad board)
At the start: 2 copper layers, 80 x 50 mm, 224 parts, among them J1 CONN_02X03, J2 CONN_02X07, J3 CONN_01X04, J4 CONN_01X01, P1 CONN_01X03, P2 CONN_01X03, P3 CONN_01X03, Q1 DMP2035U, Q2 TSM2314, Q3 DMP2035U, Q4 TSM2314, Q5 DMP2035U, Q6 TSM2314, Q7 DMP2035U, Q8 TSM2314, Q9 MMBT3904, U1 LTC6268IS8#PBF, U2 ADA4522-2ARZ, U3 ICL7660S, U4 AD8616

Commit message: Updated the glass slide holder.
Other:
- board text added: "Photodiode"
Changed lines of the file:
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@@
-(kicad_pcb (version 4) (host pcbnew 4.0.6-e0-6349~52~ubuntu17.04.1)
+(kicad_pcb (version 4) (host pcbnew 4.0.7-e0-6372~58~ubuntu17.04.1)
   (general
     (links 287)
@@
     (area 62.150001 46.15 215.357144 157.700001)
     (thickness 1.6)
-    (drawings 54)
+    (drawings 55)
     (tracks 368)
     (zones 0)
@@
     )
   )
+  (gr_text Photodiode (at 118.4 125.5) (layer Dwgs.User)
+    (effects (font (size 1.5 1.5) (thickness 0.3)))
+  )
   (dimension 50 (width 0.3) (layer Dwgs.User)
