File: pcbs/analog_board_v0.22/highCurrentPart.sch (KiCad schematic (older format))
At the start: 36 parts, among them J3 CONN_01X04, P1 CONN_01X03, P2 CONN_01X03, P3 CONN_01X03, Q1 DMP2035U, Q2 TSM2314, Q3 DMP2035U, Q4 TSM2314, Q5 DMP2035U, Q6 TSM2314, Q7 DMP2035U, Q8 TSM2314, Q9 MMBT3904, U3 ICL7660S, U4 AD8616

Commit message: Worked on the analog PCB v0.33.
Parts:
- removed 3V3, GPIO1, GPIO2, GPIO3, GPIO4, SIG1: TEST, Tespoints:TP_SMD_quadr_1mm, symbol TEST
- removed C17, C18: 10u, Resistors_SMD:R_0805, symbol C
- removed C19: 1u, Resistors_SMD:R_0805, symbol C
- removed J3: CONN_01X04, China Connectors:LED_CONN_1.25_PITCH, symbol CONN_01X04
- removed P1, P2, P3: CONN_01X03, Samtec Connectors:Samtec-PHT-1-3-01-L-S, symbol CONN_01X03
- removed Q1, Q3, Q5, Q7: DMP2035U, TO_SOT_Packages_SMD:SOT-23, symbol Q_PMOS_GSD
- removed Q2, Q4, Q6, Q8: TSM2314, TO_SOT_Packages_SMD:SOT-23, symbol Q_NMOS_GSD
- removed R10, R12: 100k, Resistors_SMD:R_0805, symbol R
- removed R11: 10k, Resistors_SMD:R_0805, symbol R
- removed RV1: T73YE103KT20, MyPotis:Vishay_T73YE103KT20, symbol POT
- removed U3: ICL7660S, SMD_Packages:SOIC-8-N, symbol ICL7660S
- removed U4: AD8616, SMD_Packages:SOIC-8-N, symbol AD8616
- added C? (x6): 10u, Resistors_SMD:R_0805, symbol C
- added J? (x4): CONN_01X02, Samtec Connectors:Samtec-PHT-1-2-01-L-S, symbol CONN_01X02
- added R?: 10k, Resistors_SMD:R_0805, symbol R
- added U? (x2): LM358, SMD_Packages:SOIC-8-N, symbol LM358
- added U? (x2): ICL7660S, SMD_Packages:SOIC-8-N, symbol ICL7660S
Connections:
- net +3V3: now also C?.1, J?.1 (P1), U?.1 (BOOST), U?.4 (V-), U?.8 (V+), U?.8 (V+)
- net +5V: no longer D2.2 (A)
- net BPW34_OUT: now also U?.1
- net GND: now also C?.2, C?.2, C?.2, C?.2, J?.2 (P2), R?.1, U?.3 (+), U?.3 (GND), U?.4 (V-), U?.5 (Vout), U?.6 (LV), U?.6 (LV), U?.8 (V+)
- net Signal: now also R?.2, U?.5 (+)
- net at Q9.1 (B): now also U?.7
- net at Q9.2 (E), R9.1: now also U?.6 (-)
- net at C23.1, D3.1 (K), R13.1: now also U?.2 (-)
- new net: C?.1, U?.2 (CAP+) (x2)
- new net: C?.2, U?.4 (CAP-) (x2)
- new net -1.65V: C?.1, J?.1 (P1), U?.5 (Vout)
- new net 1.65V: C?.1, C?.1, J?.2 (P2), U?.1 (BOOST), U?.3 (GND), U?.8 (V+)
- new net V_SENS_NEG: J?.1 (P1), J?.2 (P2)
- new net V_SENS_POS: J?.1 (P1), J?.2 (P2)
Other:
- note added: "Voltage Divider"
- note added: "Voltage Inverter"
- note removed: "Boost pin to make the oscillator faster. Enabled when connected to 3.3 V."
- note removed: "Charge pump to generate -3.3 V."
- note removed: "Constant current source with 100R sensing resistor. Monitoring diode included\nwith 1uA being translated into 1V.\n"
- note removed: "Constant current with ca. 4.55 mA."
- note removed: "H bridge for driving a coil with a rectangular signal in the mHz range. Designed\nfor at least 100 mA. Maximum current unknown."
- note removed: "Investigate if AD8616 here can be replaced by the LM358 (most likely yes, footprints match)."
- moved on the sheet: C20, C21, C22, C23, D2, D3, Q9, R13, R9
