File: pcbs/analog_board_v0.22/interface.sch (KiCad schematic (older format))
At the start: 2 parts, among them J4 CONN_02X03, J5 CONN_02X07

Commit message: Ananlog v0.33 is ready.
Parts:
- renumbered J4 to J1, J5 to J2
Connections:
- net GPIO2: now reaches J2.10 (P10)
- net GPIO1: now reaches J2.12 (P12)
- net GPIO4: now reaches J2.6 (P6)
- net GPIO3: now reaches J2.8 (P8)
- no-connect marks 8 -> 4
Changed lines of the file:
@@
 LIBS:ada4522-2
 LIBS:ltc6268
-LIBS:analog_board_v0.33-cache
+LIBS:analog_board_v0.22-cache
 EELAYER 25 0
 EELAYER END
@@
 $EndDescr
 $Comp
-L CONN_02X03 J4
+L CONN_02X03 J1
 U 1 1 5954E6D0
 P 6125 3000
-F 0 "J4" H 6125 3200 50  0000 C CNN
+F 0 "J1" H 6125 3200 50  0000 C CNN
 F 1 "CONN_02X03" H 6125 2800 50  0000 C CNN
 F 2 "Pin_Headers:Pin_Header_Angled_2x03_Pitch2.54mm" H 6125 1800 50  0001 C CNN
@@
 GND
 $Comp
-L CONN_02X07 J5
+L CONN_02X07 J2
 U 1 1 5954E8F2
 P 6125 3900
-F 0 "J5" H 6125 4300 50  0000 C CNN
+F 0 "J2" H 6125 4300 50  0000 C CNN
 F 1 "CONN_02X07" V 6125 3900 50  0000 C CNN
 F 2 "Pin_Headers:Pin_Header_Angled_2x07_Pitch2.54mm" H 6125 2700 50  0001 C CNN
@@
 NoConn ~ 5875 3800
 NoConn ~ 6375 3700
+Text HLabel 6375 3800 2    60   BiDi ~ 0
+GPIO4
+Text HLabel 6375 3900 2    60   BiDi ~ 0
+GPIO3
+Text HLabel 6375 4000 2    60   BiDi ~ 0
+GPIO2
+Text HLabel 6375 4100 2    60   BiDi ~ 0
+GPIO1
 NoConn ~ 6375 4200
-NoConn ~ 6375 3800
-NoConn ~ 6375 3900
-NoConn ~ 6375 4000
-NoConn ~ 6375 4100
 $EndSCHEMATC
