File: pcbs/analog_board_v0.22/sensitiveReadout.sch (KiCad schematic (older format))
At the start: 27 parts, among them J1 CONN_01X01, J2 CONN_01X02, J3 CONN_01X02, U1 LTC6268IS8#PBF, U2 ADA4522-2ARZ

Commit message: Ananlog v0.33 is ready.
Parts:
- removed J2, J3: CONN_01X02, Samtec Connectors:Samtec-PHT-1-2-01-L-S, symbol CONN_01X02
- removed R6: 10k, Resistors_SMD:R_0805, symbol R
- added C10: 10n, Resistors_SMD:R_0805, symbol C
- added C11, C13: 100n, Resistors_SMD:R_0805, symbol C
- added C15: 1u, Resistors_SMD:R_0805, symbol C
- added R4: 100k, Resistors_SMD:R_0805, symbol R
- added R5: 2.4k, Resistors_SMD:R_0805, symbol R
- R7: value 33k -> 1M; Farnell 2078965 -> 1576507
- renumbered C2 to C1, C10 to C12, C11 to C14, C12 to C16, C5 to C2, C7 to C3, C1 to C4, C4 to C5, C3 to C7, J1 to J4, R2 to R14, R3 to R15, R4 to R2, R5 to R3, R9 to R6
Connections:
- net V_SENS_POS is gone; now on net 3.3V: C4.1, C5.1, C6.1, U1.7 (V+)
- net GND: now also C10.2, C11.1, C13.2, C15.2; no longer U2.4 (V-)
- net at U2.1: now also R4.2, R5.1
- net at R3.1, U2.2: now also R4.1
- net at R7.2, U2.7: now also R6.1
- net +3V3 renamed 3.3V
- net BPWFA_OUT renamed BPWFA_OUT_X1
- net BPWFA_OUT_AMP renamed BPWFA_OUT_X1000
- net V_SENS_NEG renamed -3.3V
- net -3.3V: now also U2.4 (V-), C10.1, C13.1, C15.1
- new net BPWFA_OUT_X100: C11.2, R5.2
Other:
- note removed: "G = 11"
- note removed: "G = 34"
- note removed: "Gain of the second stage is selectable."
- moved on the sheet: C16, R6
