File: pcbs/backplane/backplane.sch (KiCad schematic (older format))
At the start: 57 parts, among them J1 CONN_01X04, P1 USB_B, P2 CONN_01X03, P3 CONN_02X03, P4 CONN_02X03, P5 CONN_02X07, P6 CONN_02X07, P7 CONN_01X03, P8 CONN_01X03, Q1 MMBT3904, Q2 MMBT3904, Q3 Si2323, U1 LM358, U2 TC1262-33VDB, U3 LM358, U4 CH340G, Y1 Crystal

Commit message: Added BOMs and gerber files.
Parts:
- added J2: CONN_01X01, mySamtec:Samtec-PHT-1-1-01-L-S, symbol CONN_01X01
- C6, C7: Farnell 1625484 -> 1759489
- P5, P6: Samtec (none) -> BCS-107-F-D-TE
- Q1, Q2: Farnell 1757936RL -> 2535650
Connections:
- net GND: now also J2.1 (P1)
Other:
- note added: "Grounding for the housing."

Commit message: Mechanics developed further.
Changed lines of the file:
@@
 Text GLabel 5300 2450 2    60   UnSpc ~ 0
 ADC4
-$Comp
-L CH340G U4
-U 1 1 594FA4BA
-P 5800 3950
-F 0 "U4" H 5800 3450 60  0000 C CNN
-F 1 "CH340G" H 5800 4450 60  0000 C CNN
-F 2 "SMD_Packages:SO-16-N" H 6000 3300 60  0001 C CNN
-F 3 "http://cdn2.boxtec.ch/pub/diverse/ch340g-datasheet.pdf" H 6000 3300 60  0001 C CNN
-	1    5800 3950
-	1    0    0    -1
-$EndComp
 Text GLabel 6200 1500 0    60   UnSpc ~ 0
 3.3V
@@
 	1    0    0    -1
 $EndComp
-Wire Wire Line
-	4850 1550 5400 1550
 $Comp
 L C C9
@@
 	1    0    0    1
 $EndComp
+$Comp
+L CH340G U4
+U 1 1 59610F9F
+P 5800 3950
+F 0 "U4" H 5800 3450 60  0000 C CNN
+F 1 "CH340G" H 5800 4450 60  0000 C CNN
+F 2 "SMD_Packages:SO-16-N" H 6000 3300 60  0001 C CNN
+F 3 "http://cdn2.boxtec.ch/pub/diverse/ch340g-datasheet.pdf" H 6000 3300 60  0001 C CNN
+	1    5800 3950
+	1    0    0    -1
+$EndComp
+$Comp
+L PWR_FLAG #FLG035
+U 1 1 59611BD7
+P 5100 1550
+F 0 "#FLG035" H 5100 1645 50  0001 C CNN
+F 1 "PWR_FLAG" H 5100 1730 50  0000 C CNN
+F 2 "" H 5100 1550 50  0000 C CNN
+F 3 "" H 5100 1550 50  0000 C CNN
+	1    5100 1550
+	1    0    0    -1
+$EndComp
+Wire Wire Line
+	4850 1550 5400 1550
+Connection ~ 5100 1550
 $EndSCHEMATC
