File: pcbs/analog_board_v0.33/sensitiveReadout.sch (KiCad schematic (older format))
At the start: 30 parts, among them J4 CONN_01X01, U1 LTC6268IS8#PBF, U2 ADA4522-2ARZ

Commit message: Ananlog v0.33 is ready.
Parts:
- removed C10: 10n, Resistors_SMD:R_0805, symbol C
- removed C11, C13: 100n, Resistors_SMD:R_0805, symbol C
- removed C15: 1u, Resistors_SMD:R_0805, symbol C
- removed R4: 100k, Resistors_SMD:R_0805, symbol R
- removed R5: 2.4k, Resistors_SMD:R_0805, symbol R
- added J2, J3: CONN_01X02, Samtec Connectors:Samtec-PHT-1-2-01-L-S, symbol CONN_01X02
- added R6: 10k, Resistors_SMD:R_0805, symbol R
- R7: value 1M -> 33k; Farnell 1576507 -> 2078965
- renumbered C4 to C1, C12 to C10, C14 to C11, C16 to C12, C1 to C2, C7 to C3, C5 to C4, C2 to C5, C3 to C7, J4 to J1, R14 to R2, R15 to R3, R2 to R4, R3 to R5, R6 to R9
Connections:
- net GND: now also U2.4 (V-)
- net at U2.1: now also J2.1 (P1), R6.2
- net at R5.1, U2.2: now also R6.1
- net at R7.2, U2.7: now also J2.2 (P2); no longer R9.1
- net -3.3V renamed V_SENS_NEG
- net V_SENS_NEG: no longer U2.4 (V-)
- net 3.3V renamed +3V3
- net +3V3: no longer C1.1, C4.1, C6.1, U1.7 (V+)
- net BPWFA_OUT_X1 renamed BPWFA_OUT
- net BPWFA_OUT_X1000 renamed BPWFA_OUT_AMP
- new net: J3.1 (P1), J3.2 (P2), R9.1
- new net V_SENS_POS: C1.1, C4.1, C6.1, U1.7 (V+)
Other:
- note added: "G = 11"
- note added: "G = 34"
- note added: "Gain of the second stage is selectable."
- moved on the sheet: C12, R9
