File: pcbs/analog_board_v0.33/analog_board_v0.33.kicad_pcb (KiCad board)
At the start: 2 copper layers, 80 x 50 mm, 369 parts, among them J1 CONN_01X01, J2 CONN_01X02, J3 CONN_01X02, J4 CONN_02X03, J5 CONN_02X07, J6 CONN_01X02, J7 CONN_01X02, J8 CONN_01X02, J9 CONN_01X02, Q1 MMBT3904, U1 LTC6268IS8#PBF, U2 ADA4522-2ARZ, U3 LM358, U4 ICL7660S, U5 ICL7660S

Commit message: Finished new BOM.
Connections:
- J6 pad 1: -1.65V -> GND
- J6 pad 2: GND -> -1.65V
Routing:
- net -1.65V: track 20.7 -> 17.6 mm
Other:
- board text added: "-1.65V"
- board text added: "1.65V"
- board text added: "3.3V"
- board text added: "Gain Jumper"
- board text added: "V_SENS_NEG"
- board text added: "V_SENS_POS"
- board text removed: "-1.65 V"
- board text removed: "1.65 V"
- board text removed: "3.3 V"
- board text removed: "Gain Jumpers"
Changed lines of the file:
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@@
     (area 62.150001 46.15 215.357144 157.700001)
     (thickness 1.6)
-    (drawings 46)
-    (tracks 259)
+    (drawings 48)
+    (tracks 257)
     (zones 0)
     (modules 369)
@@
   )
   (setup
-    (last_trace_width 0.25)
+    (last_trace_width 0.4)
     (user_trace_width 0.4)
     (trace_clearance 0.2)
@@
     (fp_line (start 1.6 -1.6) (end -1.6 -1.6) (layer F.CrtYd) (width 0.05))
     (pad 1 thru_hole rect (at 0 0) (size 2 2) (drill 1.2) (layers *.Cu *.Mask)
-      (net 21 -1.65V))
-    (pad 2 thru_hole oval (at 0 2.54) (size 2 2) (drill 1.2) (layers *.Cu *.Mask)
       (net 1 GND))
+    (pad 2 thru_hole oval (at 0 2.54) (size 2 2) (drill 1.2) (layers *.Cu *.Mask)
+      (net 21 -1.65V))
     (model Pin_Headers.3dshapes/Pin_Header_Straight_1x02_Pitch2.54mm.wrl
       (at (xyz 0 -0.05 0))
@@
       (net 7 Signal))
   )
-  (gr_text GND (at 149.098 129.794) (layer F.SilkS)
+  (gr_text V_SENS_NEG (at 155.829 122.682) (layer F.SilkS)
+    (effects (font (size 1.5 1.5) (thickness 0.3)))
+  )
+  (gr_text V_SENS_POS (at 155.829 112.268) (layer F.SilkS)
+    (effects (font (size 1.5 1.5) (thickness 0.3)))
+  )
+  (gr_text GND (at 148.59 129.667) (layer F.SilkS)
     (effects (font (size 1.5 1.5) (thickness 0.3)))
   )
-  (gr_text "-1.65 V" (at 146.685 127) (layer F.SilkS)
+  (gr_text -1.65V (at 146.685 127) (layer F.SilkS)
     (effects (font (size 1.5 1.5) (thickness 0.3)))
   )
-  (gr_text "1.65 V" (at 147.701 119.38) (layer F.SilkS)
+  (gr_text 1.65V (at 147.701 119.38) (layer F.SilkS)
     (effects (font (size 1.5 1.5) (thickness 0.3)))
   )
-  (gr_text "3.3 V" (at 148.463 116.84) (layer F.SilkS)
+  (gr_text 3.3V (at 148.463 116.84) (layer F.SilkS)
     (effects (font (size 1.5 1.5) (thickness 0.3)))
   )
@@
     (effects (font (size 1.5 1.5) (thickness 0.3)))
   )
-  (gr_text "Gain Jumpers" (at 129.921 88.9) (layer F.SilkS)
+  (gr_text "Gain Jumper" (at 129.921 88.9) (layer F.SilkS)
     (effects (font (size 1.5 1.5) (thickness 0.3)))
   )
@@
   (segment (start 165.608 118.872) (end 168.783 118.872) (width 0.4) (layer F.Cu) (net 20))
   (segment (start 168.783 118.872) (end 168.844 118.811) (width 0.25) (layer F.Cu) (net 20))
-  (segment (start 155.448 127) (end 157.607 127) (width 0.4) (layer F.Cu) (net 21))
-  (segment (start 168.656 130.937) (end 168.656 130.175) (width 0.4) (layer F.Cu) (net 21))
-  (segment (start 167.64 131.953) (end 168.656 130.937) (width 0.4) (layer F.Cu) (net 21))
-  (segment (start 159.131 131.953) (end 167.64 131.953) (width 0.4) (layer F.Cu) (net 21))
-  (segment (start 158.242 131.064) (end 159.131 131.953) (width 0.4) (layer F.Cu) (net 21))
-  (segment (start 158.242 127.635) (end 158.242 131.064) (width 0.4) (layer F.Cu) (net 21))
-  (segment (start 157.607 127) (end 158.242 127.635) (width 0.4) (layer F.Cu) (net 21))
+  (segment (start 168.656 130.175) (end 168.656 130.556) (width 0.4) (layer F.Cu) (net 21))
+  (segment (start 155.448 130.556) (end 155.448 129.54) (width 0.4) (layer F.Cu) (net 21))
+  (segment (start 156.337 131.445) (end 155.448 130.556) (width 0.4) (layer F.Cu) (net 21))
+  (segment (start 167.767 131.445) (end 156.337 131.445) (width 0.4) (layer F.Cu) (net 21))
+  (segment (start 168.656 130.556) (end 167.767 131.445) (width 0.4) (layer F.Cu) (net 21))
   (segment (start 170.815 130.368) (end 168.849 130.368) (width 0.4) (layer F.Cu) (net 21))
   (segment (start 168.849 130.368) (end 168.656 130.175) (width 0.4) (layer F.Cu) (net 21))
